Commit message: update

File: dev_ws/src/rm_gimbal_description/urdf/rm_gimbal.urdf.xacro (robot description, xacro)
@@ -13,4 +13,5 @@
   <joint name="camera_joint" type="fixed">
     <origin xyz="$(arg xyz)" rpy="$(arg rpy)" />
+<!--    <origin xyz="0 0 0" rpy="0 0 0" />-->
     <parent link="gimbal_link" />
     <child link="camera_link" />
